File: HOPE_Project.sch (KiCad schematic (older format))
At the start: 26 parts, among them J1 Serial_to_USB, J2 LCD_Screen, U1 V7805-1000, U2 ATmega168A-PU, Y1 Crystal

Commit message: Finish board
Parts:
- RV1: footprint Resistor_SMD:R_0201_0603Metric -> digikey-footprints:Potentiometer_P120PK-Y25BR10K
- Y1: footprint Crystal:Crystal_HC49-U_Horizontal -> Crystal:Crystal_HC49-U_Vertical
Connections:
- net GND: now also R3.2
Changed lines of the file:
@@
 F 0 "RV1" H 8331 3204 50  0000 R CNN
 F 1 "10 kOhm" H 8331 3295 50  0000 R CNN
-F 2 "Resistor_SMD:R_0201_0603Metric" H 8400 3250 50  0001 C CNN
+F 2 "digikey-footprints:Potentiometer_P120PK-Y25BR10K" H 8400 3250 50  0001 C CNN
 F 3 "~" H 8400 3250 50  0001 C CNN
 	1    8400 3250
@@
 F 0 "Y1" V 4204 3181 50  0000 L CNN
 F 1 "Crystal" V 4295 3181 50  0000 L CNN
-F 2 "Crystal:Crystal_HC49-U_Horizontal" H 4250 3050 50  0001 C CNN
+F 2 "Crystal:Crystal_HC49-U_Vertical" H 4250 3050 50  0001 C CNN
 F 3 "~" H 4250 3050 50  0001 C CNN
 	1    4250 3050
@@
 L power:GND #PWR0126
 U 1 1 5CA56AF2
-P 6500 6100
-F 0 "#PWR0126" H 6500 5850 50  0001 C CNN
-F 1 "GND" H 6505 5927 50  0000 C CNN
-F 2 "" H 6500 6100 50  0001 C CNN
-F 3 "" H 6500 6100 50  0001 C CNN
-	1    6500 6100
-	1    0    0    -1
-$EndComp
+P 6500 6050
+F 0 "#PWR0126" H 6500 5800 50  0001 C CNN
+F 1 "GND" H 6505 5877 50  0000 C CNN
+F 2 "" H 6500 6050 50  0001 C CNN
+F 3 "" H 6500 6050 50  0001 C CNN
+	1    6500 6050
+	1    0    0    -1
+$EndComp

Commit message: First round of adjustments
Parts:
- removed J1: Serial_to_USB, HOPE_Project:Serial_Breakout, symbol Connector:Conn_01x06_Male
- added C5: 100 nF, Capacitor_SMD:C_0201_0603Metric, symbol Device:C
- added C6: 100 uF, Capacitor_SMD:C_1206_3216Metric, symbol Device:C
- added D2: D_Schottky, Diode_SMD:D_SOD-323, symbol Device:D_Schottky
- added R8: 10 kOhm, Resistor_SMD:R_0201_0603Metric, symbol Device:R
- added S6: EG1903-ND, digikey-footprints:Switch_Slide_11.6x4mm_EG1218, symbol EG1903-ND:EG1903-ND
- added S7: KS-01Q-01, digikey-footprints:PushButton_Round_D12mm_THT_KS-01Q-01, symbol dk_Pushbutton-Switches:KS-01Q-01
- R2, R3, R5, R6: value 1 kOhm -> 10 kOhm
Connections:
- net +5V: now also C5.1, C6.1, S6.3, S7.2; no longer C2.1, U1.3 (Vo+)
- net A1: now also S5.3; no longer S3.3
- net A3: now also S7.3; no longer S5.3
- net GND: now also C5.2, C6.2, D2.2 (A), R8.2
- net A4: now reaches U2.27 (PC4)
- net A4: now also S3.3
- net at BT1.1 (+), C1.1, U1.1 (Vin+): now also D2.1 (K)
- net RX: no longer names the net of U2.2 (PD0)
- net TX: no longer names the net of U2.3 (PD1)
- new net: C2.1, S6.2, U1.3 (Vo+)
- new net: R8.1, S7.1
Other:
- moved on the sheet: D1, R7
